File: hardware/MDC.kicad_sch (KiCad schematic)
At the start: 31 parts, among them J1 USB_C_Receptacle_USB2.0_16P, J2 SWD Debug Header, J3 Conn_01x20, J4 Conn_01x20, SW1 BOOTSEL_Button, SW2 Reset_Button, U1 RP2040, U2 W25Q128JVS, U3 AP2112K-3.3, U4 USBLC6-2SC6, Y1 Crystal_GND24_Small

Commit message: Chore: MDC-backups klasörü git takibinden çıkarıldı
Other:
- note added: "Connectors"
- note added: "Flash Memory"
- note added: "Microcontroller"
- note added: "Power LED"
- note added: "USB Interface"
- note added: "USB-C"
- company: (none) -> TURQON
- title: (none) -> MDC RP2040 Minimal Dev Board
- moved on the sheet: C1, C12, C13, C2, C3, C4, C5, C6, D1, D2, J1, J2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
